File: hardware/okey.kicad_pcb (KiCad board)
At the start: 2 copper layers, 243.8 x 352.4 mm, 150 parts, among them IC1 4094N, IC2 4094N, P1 ROW_JMP, P10 CONN_02X06, P11 CONN_02X06, P12 CONN_02X06, P13 CONN_02X06, P14 CONN_02X06, P15 CONN_02X06, P16 CONN_02X08, P17 CONN_01X01, P18 CONN_02X08, P19 CONN_01X01, P2 CONN_02X13, P20 CONN_01X01, P21 CONN_01X01, P22 CONN_02X08, P23 CONN_02X08, P24 CONN_02X06, P25 CONN_02X06, P26 CONN_02X06, P27 CONN_02X06, P28 CONN_02X06, P29 CONN_02X06, P3 CONN_02X03, P30 CONN_02X08, P31 CONN_02X03, P32 CONN_02X03, P33 CONN_02X06, P34 CONN_02X06, P35 CONN_02X06, P36 CONN_02X06, P37 CONN_02X06, P38 CONN_02X06, P39 CONN_01X01, P4 CONN_02X08, P40 CONN_02X03, P41 CONN_02X06, P42 CONN_02X06, P43 CONN_02X06, P44 CONN_02X06, P45 CONN_02X06, P46 CONN_02X06, P47 CONN_01X01, P5 CONN_02X03, P6 CONN_02X10, P7 CONN_02X03, P8 CONN_01X01, P9 CONN_02X08, Q1 Q_NPN_BCE, Q2 Q_NPN_BCE, Q3 Q_NPN_BCE, SW1 MX_D, SW10 MX_D, SW11 MX_D, SW12 MX_D, SW13 MX_D, SW14 MX_D, SW15 MX_D, SW16 MX_D, SW17 MX_D, SW18 MX_D, SW19 SW_PUSH, SW2 MX_D, SW20 SW_PUSH, SW21 SW_PUSH, SW22 SW_PUSH, SW23 SW_PUSH, SW24 SW_PUSH, SW25 SW_PUSH, SW26 SW_PUSH, SW27 SW_PUSH, SW28 SW_PUSH, SW29 SW_PUSH, SW3 MX_D, SW30 SW_PUSH, SW31 SW_PUSH, SW32 SW_PUSH, SW33 SW_PUSH, SW34 SW_PUSH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

Commit message: hardware: add bypass capacitors
Parts:
- added C1: 1uF, Capacitors_ThroughHole:CP_Radial_Tantal_D5.0mm_P2.50mm, F.Cu at (90.2, 24.1)
- added C2: 100nF, Capacitors_ThroughHole:CP_Radial_Tantal_D5.0mm_P2.50mm, F.Cu at (87.6, 33.0)
- added C3: 100nF, Capacitors_ThroughHole:CP_Radial_Tantal_D5.0mm_P2.50mm, F.Cu at (52.1, 31.8)
- added C4: 100nF, Capacitors_ThroughHole:CP_Radial_Tantal_D5.0mm_P2.50mm, F.Cu at (55.9, 66.0)
- added C5: 100nF, Capacitors_ThroughHole:CP_Radial_Tantal_D5.0mm_P2.50mm, F.Cu at (36.8, 66.0)
- added C6, C7: 100nF, Capacitors_ThroughHole:CP_Radial_Tantal_D5.0mm_P2.50mm, F.Cu at (91.4, 73.7)
- COL_SELECT1, COL_SELECT2, COL_SELECT3, COL_SELECT4, P16, P18, P22, P23, P30, P4, P9: footprint Pin_Headers:Pin_Header_Straight_2x08 -> Pin_Headers:Pin_Header_Straight_2x08_Pitch2.54mm
- IC1, IC2: footprint Housings_DIP:DIP-16_W7.62mm_LongPads -> Housings_DIP:DIP-16_W7.62mm
- P1, P2: footprint Pin_Headers:Pin_Header_Straight_2x13 -> Pin_Headers:Pin_Header_Straight_2x13_Pitch2.54mm
- P10, P11, P12, P13, P14, P15, P24, P25, P26, P27, P28, P29: footprint Pin_Headers:Pin_Header_Straight_2x06 -> Pin_Headers:Pin_Header_Straight_2x06_Pitch2.54mm
- P17, P19, P20, P21, P8: footprint Pin_Headers:Pin_Header_Straight_1x01 -> Pin_Headers:Pin_Header_Straight_1x01_Pitch2.54mm
- P3, P31, P5, P7: footprint Pin_Headers:Pin_Header_Straight_2x03 -> Pin_Headers:Pin_Header_Straight_2x03_Pitch2.54mm
- P6: footprint Pin_Headers:Pin_Header_Straight_2x10 -> Pin_Headers:Pin_Header_Straight_2x10_Pitch2.54mm
- PNL_ID1: footprint Pin_Headers:Pin_Header_Straight_2x07 -> Pin_Headers:Pin_Header_Straight_2x07_Pitch2.54mm
- ROW_SELECT1, ROW_SELECT2: footprint Pin_Headers:Pin_Header_Straight_1x08 -> Pin_Headers:Pin_Header_Straight_1x08_Pitch2.54mm
- moved P3 2.54 mm to (92.7, 22.9)
Routing:
- net GND: track 395.5 -> 421.6 mm, vias 4 -> 5
- net VDD: track 423.1 -> 437.5 mm
- net Net-(IC2-Pad4): track 31.9 -> 38.5 mm
- net Net-(IC2-Pad5): track 33.4 -> 40.0 mm
- net Net-(IC2-Pad6): track 34.2 -> 40.7 mm
- net Net-(IC1-Pad9): track 64.5 -> 71.1 mm
- net Net-(IC2-Pad7): track 32.7 -> 36.7 mm
- net Net-(P3-Pad4): track 20.9 -> 24.7 mm
- net Net-(P3-Pad1): track 232.1 -> 234.8 mm
- net Net-(IC1-Pad2): track 60.2 -> 62.7 mm
- net Net-(P3-Pad6): track 16.6 -> 18.8 mm
- net Net-(D7-Pad2): track 93.1 -> 94.6 mm
- net Net-(MUX_COL1-Pad9): track 24.0 -> 25.5 mm
- net Net-(MUX_COL1-Pad10): track 23.0 -> 23.7 mm

Commit message: hardware: rework SPI board as SMD board with smaller dimensions ...
Parts:
- added P48: CONN_02X03, Pin_Headers:Pin_Header_Straight_2x03_Pitch2.54mm, F.Cu at (99.1, 43.2)
- D1, D2, D3, D4, D5, D6, D7, D8: footprint Resistors_ThroughHole:Resistor_Horizontal_RM15mm -> Discret:CP6
- D10, D11, D12, D13, D14, D15, D16, D17, D18, D19, D20, D21, D22, D23, D24, D9: footprint Discret:D4 -> Discret:R4
- IC1, IC2, MUX_COL1, MUX_ROW1, U1: footprint Housings_DIP:DIP-16_W7.62mm -> Housings_SSOP:SOP-16_4.4x10.4mm_Pitch1.27mm; moved to B.Cu
- U2: footprint Housings_DIP:DIP-14_W7.62mm -> Housings_SOIC:SOIC-14_3.9x8.7mm_Pitch1.27mm; moved to B.Cu
- moved MUX_COL1 56.5 mm to (114.3, 41.3), turned to 180 degrees
- moved C3 46.1 mm to (64.1, 76.2)
- moved C4 42.4 mm to (22.9, 39.4), turned to 270 degrees
- moved D10 40.7 mm to (184.2, 88.9)
- moved D14 40.7 mm to (205.7, 88.9)
- moved D15 40.7 mm to (215.9, 78.7)
- moved D19 40.7 mm to (241.3, 78.7)
- moved D20 40.7 mm to (243.8, 88.9)
- moved D22 40.7 mm to (256.5, 88.9)
- moved D24 40.7 mm to (265.4, 88.9)
- moved D25 40.7 mm to (212.1, 19.1)
- moved D9 40.7 mm to (181.6, 78.7)
- moved P31 40.7 mm to (198.1, 26.7)
- moved Q1 40.7 mm to (194.3, 36.8)
- moved Q2 40.7 mm to (194.3, 41.9)
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Routing:
- net VDD: track 437.5 -> 111.5 mm, vias 2 -> 1
- net GND: track 421.6 -> 118.4 mm, vias 5 -> 2
- net Net-(MUX_COL1-Pad3): track 226.0 -> 45.7 mm
- net Net-(P3-Pad1): track 234.8 -> 54.8 mm
- net Net-(IC1-Pad1): track 250.2 -> 124.6 mm, vias 0 -> 2
- net Net-(IC1-Pad3): track 226.4 -> 105.2 mm
- net Net-(D23-Pad2): track 119.8 -> 26.5 mm
- net Net-(D23-Pad1): track 7.40 -> 96.7 mm
- net Net-(D17-Pad2): track 115.6 -> 36.8 mm
- net Net-(D7-Pad2): track 94.6 -> 24.8 mm
- net Net-(D19-Pad2): track 117.1 -> 57.3 mm
- net Net-(MUX_ROW1-Pad11): track 73.3 -> 14.7 mm
- net Net-(D8-Pad2): track 92.4 -> 34.6 mm
- net Net-(D21-Pad1): track 7.40 -> 64.1 mm
- net Net-(D21-Pad2): track 118.0 -> 61.3 mm
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Other:
- board size 243.8 x 352.4 mm -> 263.4 x 349.9 mm
